Commit message: updated model first time

File: urdf/Robot_URDF.urdf (robot description, URDF)
Before this commit: robot Robot_URDF, 5 links, 4 joints
Links:
- link Back_Left: mass 0.011306 -> 0.0113055466168378
- link Back_Right: mass 0.011306 -> 0.0113055466168378
- link Front_Left: mass 0.011306 -> 0.0113055466168378
- link Front_Right: mass 0.011306 -> 0.0113055466168378

Commit message: added wheels, set coordinate frames

File: urdf/Robot_URDF.urdf (robot description, URDF)
Before this commit: robot Robot_URDF, 5 links, 4 joints
Links:
- removed link Back_Left
- removed link Back_Right
- removed link Front_Left
- removed link Front_Right
- added link w_front_left, mass 2.1167; collision mesh filename=package://robot_urdf/meshes/w_front_left.STL; visual mesh filename=package://robot_urdf/meshes/w_front_left.STL
- added link w_front_right, mass 2.1167; collision mesh filename=package://robot_urdf/meshes/w_front_right.STL; visual mesh filename=package://robot_urdf/meshes/w_front_right.STL
- added link w_rear_left, mass 2.1167; collision mesh filename=package://robot_urdf/meshes/w_rear_left.STL; visual mesh filename=package://robot_urdf/meshes/w_rear_left.STL
- added link w_rear_right, mass 2.1167; collision mesh filename=package://robot_urdf/meshes/w_rear_right.STL; visual mesh filename=package://robot_urdf/meshes/w_rear_right.STL
- link base_link: mass 0.192303858587445 -> 24.944; geometry collision mesh filename=package://robot_urdf/meshes/base_link.STL; visual mesh filename=package://robot_urdf/meshes/base_link.STL
Joints:
- removed joint Back_Left_Joint
- removed joint Back_Right_Joint
- removed joint Front_Left_joint
- removed joint Front_Right_Joint
- added joint j_front_left: type revolute, parent base_link, child w_front_left, origin xyz=0 0 0 rpy=0 0 0, axis 0 1 0, limit lower=0 upper=0 effort=30 velocity=30
- added joint j_front_right: type revolute, parent base_link, child w_front_right, origin xyz=0 0 0 rpy=0 0 0, axis 0 -1 0, limit lower=0 upper=0 effort=0 velocity=0
- added joint j_rear_left: type revolute, parent base_link, child w_rear_left, origin xyz=0 0 0 rpy=0 0 0, axis 0 1 0, limit lower=0 upper=0 effort=0 velocity=0
- added joint j_rear_right: type revolute, parent base_link, child w_rear_right, origin xyz=0 0 0 rpy=0 0 0, axis 0 -1 0, limit lower=0 upper=0 effort=0 velocity=0
