Commit message: Corrected some lidar files, Added World file
Sanitized the repository
Corrected ydlidar.urdf
Added competition arena.world file
Added xacro file in the correct folder

File: urdf/ydlidar.urdf (robot description, URDF)
Before this commit: robot ydlidar, 2 links, 1 joints
Links:
- link base_laser: geometry collision mesh filename=package://robot_urdf/meshes/ydlidar.dae; visual mesh filename=package://robot_urdf/meshes/ydlidar.dae
