Commit message: Redesigned Robot

File: urdf/robot_urdf.urdf (robot description, URDF)
Before this commit: robot robot_urdf, 6 links, 5 joints
Links:
- removed link dummy_link
- removed link w_front_left
- removed link w_front_right
- removed link w_rear_left
- removed link w_rear_right
- added link front_left_chassis, mass 0.141762199312227; collision mesh filename=package://robot_urdf/meshes/front_left_chassis.STL; visual mesh filename=package://robot_urdf/meshes/front_left_chassis.STL
- added link front_left_wheel, mass 5.71507847538441; collision mesh filename=package://robot_urdf/meshes/front_left_wheel.STL; visual mesh filename=package://robot_urdf/meshes/front_left_wheel.STL
- added link front_right_chassis, mass 0.141762199312227; collision mesh filename=package://robot_urdf/meshes/front_right_chassis.STL; visual mesh filename=package://robot_urdf/meshes/front_right_chassis.STL
- added link front_right_wheel, mass 5.71507847538429; collision mesh filename=package://robot_urdf/meshes/front_right_wheel.STL; visual mesh filename=package://robot_urdf/meshes/front_right_wheel.STL
- added link rear_left_wheel, mass 5.71507847538442; collision mesh filename=package://robot_urdf/meshes/rear_left_wheel.STL; visual mesh filename=package://robot_urdf/meshes/rear_left_wheel.STL
- added link rear_right_wheel, mass 5.71507847538443; collision mesh filename=package://robot_urdf/meshes/rear_right_wheel.STL; visual mesh filename=package://robot_urdf/meshes/rear_right_wheel.STL
- link base_link: mass 24.944 -> 50.9630293132178
Joints:
- removed joint dummy_joint
- removed joint j_front_left
- removed joint j_front_right
- removed joint j_rear_left
- removed joint j_rear_right
- added joint j_front_left_chassis: type revolute, parent base_link, child front_left_chassis, origin xyz=0 -0.0381 0 rpy=1.5708 0 0, axis 0 0 1, limit lower=0 upper=0 effort=0 velocity=0
- added joint j_front_left_wheel: type revolute, parent front_left_chassis, child front_left_wheel, origin xyz=0 0 0 rpy=0 0 0, axis -0.318646885836196 -0.947873494801334 0, limit lower=0 upper=0 effort=0 velocity=0
- added joint j_front_right_chassis: type revolute, parent base_link, child front_right_chassis, origin xyz=0 -0.0381 0 rpy=1.5707963267949 0 0, axis 0 0 1, limit lower=0 upper=0 effort=0 velocity=0
- added joint j_front_right_wheel: type continuous, parent front_right_chassis, child front_right_wheel, origin xyz=0 0 0 rpy=0 0 0, axis 0.357981701084848 -0.93372860172986 0
- added joint j_rear_left_wheel: type revolute, parent base_link, child rear_left_wheel, origin xyz=0 -0.0381 0 rpy=1.5708 0 0, axis 0 1 0, limit lower=0 upper=0 effort=0 velocity=0
- added joint j_rear_right_wheel: type revolute, parent base_link, child rear_right_wheel, origin xyz=0 -0.0381 0 rpy=1.5708 0 0, axis 0 1 0, limit lower=0 upper=0 effort=0 velocity=0

Commit message: Gains Added
Added Gains
Correct robot_urdf

File: urdf/robot_urdf.urdf (robot description, URDF)
Before this commit: robot robot_urdf, 7 links, 6 joints
Joints:
- joint j_rear_left_wheel: limit (none) -> effort=30 velocity=100
- joint j_support_right: limit lower=-1.0472 upper=1.0472 effort=30 velocity=100 -> lower=-1.0472 upper=1.0472 effort=10 velocity=100
