Commit message: Updated launch files, redid changes on CMakeList,Package.xml

File: urdf/integrated2.urdf (robot description, URDF)
Before this commit: robot robot_urdf, 8 links, 7 joints
Joints:
- joint sensor_joint: origin xyz=0.45 0 0.09 rpy=3.14 0 3.14 -> xyz=0.45 0 0.09 rpy=0 0 0

File: xacro/robot.xacro (robot description, xacro)
@@ -39,5 +39,5 @@
             <plugin name="gazebo_ros_head_hokuyo_controller" filename="libgazebo_ros_laser.so">
             	<!-- Use topic name as /my_robot/scan -->
-				<topicName></topicName>
+				<topicName>/robot_urdf/laser_scan</topicName>
 				<frameName>laser_frame</frameName>
 			</plugin>
@@ -45,5 +45,5 @@
 	</gazebo>
 <!--  Gazebo plugin for control here is already added for you -->
-	<gazebo>
+	<!-- <gazebo>
 		<plugin name="gazebo_ros_control" filename="libgazebo_ros_control.so">
 			<robotNamespace>/robot_urdf</robotNamespace>
@@ -51,9 +51,12 @@
 			<legacyModeNS>true</legacyModeNS>
 		</plugin>
-	</gazebo>
+	</gazebo> -->
 <!-- Create a joint between your robot and sensor -->
 	<joint
-    name="sensor_joint"
-    type="fixed">
+      name="sensor_joint"
+      type="fixed">
+	  <origin
+		  xyz="0.45 0 0.09"
+		  rpy="0 0 0" />
     <parent
       link="dummy_link" />
@@ -61,3 +64,33 @@
       link="base_laser" />
 	</joint>
+	<!-- <material name="red">
+		<color rgba="0.8 0.0 0.0 1.0"/>
+	</material>
+	<material name="black">
+		<color rgba="0.0 0.0 0.0 1.0"/>
+	</material>
+	<material name="dark">
+		<color rgba="0.3 0.3 0.3 1.0"/>
+	</material>
+	<gazebo reference="base_link">
+		<material>Gazebo/Red</material>
+	</gazebo>
+	<gazebo reference="w_rear_right">
+		<material>Gazebo/FlatBlack</material>
+	</gazebo>
+	<gazebo reference="w_rear_left">
+		<material>Gazebo/FlatBlack</material>
+	</gazebo>
+	<gazebo reference="w_front_right">
+		<material>Gazebo/FlatBlack</material>
+	</gazebo>
+	<gazebo reference="w_front_left">
+		<material>Gazebo/FlatBlack</material>
+	</gazebo>
+	<link name="dummy_link">
+	</link>
+	<joint name="dummy_joint" type="fixed">
+		<parent link="dummy_link"/>
+		<child link="base_link"/>
+	</joint> -->
 </robot>

Commit message: Model resdesign successful

File: urdf/integrated2.urdf (robot description, URDF)
Before this commit: robot robot_urdf, 8 links, 7 joints
Links:
- removed link w_front_left
- removed link w_front_right
- removed link w_rear_left
- removed link w_rear_right
- added link front_left_wheel, mass 5.71507847538447; collision mesh filename=package://robot_urdf/meshes/front_left_wheel.STL; visual mesh filename=package://robot_urdf/meshes/front_left_wheel.STL
- added link front_right_wheel, mass 5.71507847538445; collision mesh filename=package://robot_urdf/meshes/front_right_wheel.STL; visual mesh filename=package://robot_urdf/meshes/front_right_wheel.STL
- added link rear_left_wheel, mass 5.71507847538444; collision mesh filename=package://robot_urdf/meshes/rear_left_wheel.STL; visual mesh filename=package://robot_urdf/meshes/rear_left_wheel.STL
- added link rear_right_wheel, mass 5.71507847538442; collision mesh filename=package://robot_urdf/meshes/rear_right_wheel.STL; visual mesh filename=package://robot_urdf/meshes/rear_right_wheel.STL
- added link support_left, mass 0.141762199312228; collision mesh filename=package://robot_urdf/meshes/support_left.STL; visual mesh filename=package://robot_urdf/meshes/support_left.STL
- added link support_right, mass 0.141762199312228; collision mesh filename=package://robot_urdf/meshes/support_right.STL; visual mesh filename=package://robot_urdf/meshes/support_right.STL
- link base_link: mass 24.944 -> 51.1408666026729
Joints:
- removed joint j_front_left
- removed joint j_front_right
- removed joint j_rear_left
- removed joint j_rear_right
- added joint j_front_left_wheel: type continuous, parent support_left, child front_left_wheel, origin xyz=0 -0.0299999999999973 -0.14732 rpy=1.5707963267949 0 0, axis 0 0 -1, limit lower=0 upper=0 effort=0 velocity=0
- added joint j_front_right_wheel: type continuous, parent support_right, child front_right_wheel, origin xyz=0 -0.0299999999999997 -0.14732 rpy=1.5707963267949 0 0, axis 0 0 -1, limit lower=0 upper=0 effort=0 velocity=0
- added joint j_rear_left_wheel: type continuous, parent base_link, child rear_left_wheel, origin xyz=-0.3683 0.18113 0.11557 rpy=1.5707963267949 0 0, axis 0 0 1
- added joint j_rear_right_wheel: type continuous, parent base_link, child rear_right_wheel, origin xyz=-0.3683 -0.18113 0.11557 rpy=1.5707963267949 0 0, axis 0 0 1, limit lower=0 upper=0 effort=0 velocity=0
- added joint j_support_left: type continuous, parent base_link, child support_left, origin xyz=0.368299999999998 0.152399999999998 0.26289 rpy=0 0 0, axis 0 0 1, limit lower=0 upper=0 effort=0 velocity=0
- added joint j_support_right: type continuous, parent base_link, child support_right, origin xyz=0.3683 -0.1524 0.26289 rpy=0 0 0, axis 0 0 1, limit lower=0 upper=0 effort=0 velocity=0

File: urdf/robot_urdf.urdf (robot description, URDF)
Before this commit: robot robot_urdf, 7 links, 6 joints
Links:
- removed link front_left_chassis
- removed link front_right_chassis
- added link support_left, mass 0.141762199312228; collision mesh filename=package://robot_urdf/meshes/support_left.STL; visual mesh filename=package://robot_urdf/meshes/support_left.STL
- added link support_right, mass 0.141762199312228; collision mesh filename=package://robot_urdf/meshes/support_right.STL; visual mesh filename=package://robot_urdf/meshes/support_right.STL
- link base_link: mass 50.9630293132178 -> 51.1408666026729
- link front_left_wheel: mass 5.71507847538441 -> 5.71507847538447
- link front_right_wheel: mass 5.71507847538429 -> 5.71507847538445
- link rear_left_wheel: mass 5.71507847538442 -> 5.71507847538444
- link rear_right_wheel: mass 5.71507847538443 -> 5.71507847538442
Joints:
- removed joint j_front_left_chassis
- removed joint j_front_right_chassis
- added joint j_support_left: type continuous, parent base_link, child support_left, origin xyz=0.368299999999998 0.152399999999998 0.26289 rpy=0 0 0, axis 0 0 1, limit lower=0 upper=0 effort=0 velocity=0
- added joint j_support_right: type continuous, parent base_link, child support_right, origin xyz=0.3683 -0.1524 0.26289 rpy=0 0 0, axis 0 0 1, limit lower=0 upper=0 effort=0 velocity=0
- joint j_front_left_wheel: axis -0.318646885836196 -0.947873494801334 0 -> 0 0 -1; origin xyz=0 0 0 rpy=0 0 0 -> xyz=0 -0.0299999999999973 -0.14732 rpy=1.5707963267949 0 0; parent front_left_chassis -> support_left; type revolute -> continuous
- joint j_front_right_wheel: axis 0.357981701084848 -0.93372860172986 0 -> 0 0 -1; limit (none) -> lower=0 upper=0 effort=0 velocity=0; origin xyz=0 0 0 rpy=0 0 0 -> xyz=0 -0.0299999999999997 -0.14732 rpy=1.5707963267949 0 0; parent front_right_chassis -> support_right
- joint j_rear_left_wheel: axis 0 1 0 -> 0 0 1; limit lower=0 upper=0 effort=0 velocity=0 -> (none); origin xyz=0 -0.0381 0 rpy=1.5708 0 0 -> xyz=-0.3683 0.18113 0.11557 rpy=1.5707963267949 0 0; type revolute -> continuous
- joint j_rear_right_wheel: axis 0 1 0 -> 0 0 1; origin xyz=0 -0.0381 0 rpy=1.5708 0 0 -> xyz=-0.3683 -0.18113 0.11557 rpy=1.5707963267949 0 0; type revolute -> continuous

File: xacro/robot.xacro (robot description, xacro)
@@ -64,5 +64,5 @@
       link="base_laser" />
 	</joint>
-	<!-- <material name="red">
+	<material name="red">
 		<color rgba="0.8 0.0 0.0 1.0"/>
 	</material>
@@ -76,5 +76,5 @@
 		<material>Gazebo/Red</material>
 	</gazebo>
-	<gazebo reference="w_rear_right">
+	<!-- <gazebo reference="w_rear_right">
 		<material>Gazebo/FlatBlack</material>
 	</gazebo>
@@ -87,5 +87,5 @@
 	<gazebo reference="w_front_left">
 		<material>Gazebo/FlatBlack</material>
-	</gazebo>
+	</gazebo> -->
 	<link name="dummy_link">
 	</link>
@@ -93,4 +93,4 @@
 		<parent link="dummy_link"/>
 		<child link="base_link"/>
-	</joint> -->
+	</joint>
 </robot>

Commit message: Fixed link colors, fixed lidar position

File: urdf/integrated2.urdf (robot description, URDF)
Before this commit: robot robot_urdf, 10 links, 9 joints
Joints:
- joint sensor_joint: origin xyz=0.45 0 0.09 rpy=0 0 0 -> xyz=0.44 0 0.275 rpy=0 0 0

File: xacro/robot.xacro (robot description, xacro)
@@ -57,5 +57,5 @@
       type="fixed">
 	  <origin
-		  xyz="0.45 0 0.09"
+		  xyz="0.44 0 0.275"
 		  rpy="0 0 0" />
     <parent
@@ -76,16 +76,22 @@
 		<material>Gazebo/Red</material>
 	</gazebo>
-	<!-- <gazebo reference="w_rear_right">
+	<gazebo reference="support_left">
+		<material>Gazebo/Red</material>
+	</gazebo>
+	<gazebo reference="support_right">
+		<material>Gazebo/Red</material>
+	</gazebo>
+	<gazebo reference="front_left_wheel">
 		<material>Gazebo/FlatBlack</material>
 	</gazebo>
-	<gazebo reference="w_rear_left">
+	<gazebo reference="front_right_wheel">
 		<material>Gazebo/FlatBlack</material>
 	</gazebo>
-	<gazebo reference="w_front_right">
+	<gazebo reference="rear_left_wheel">
 		<material>Gazebo/FlatBlack</material>
 	</gazebo>
-	<gazebo reference="w_front_left">
+	<gazebo reference="rear_right_wheel">
 		<material>Gazebo/FlatBlack</material>
-	</gazebo> -->
+	</gazebo>
 	<link name="dummy_link">
 	</link>

Commit message: Added transmission and Controllers for joints
Added sane joint limits
Front wheel steering joints are revolute with +-60 deg limits

File: urdf/integrated2.urdf (robot description, URDF)
Before this commit: robot robot_urdf, 10 links, 9 joints
Joints:
- joint j_front_left_wheel: limit lower=0 upper=0 effort=0 velocity=0 -> effort=30 velocity=100
- joint j_front_right_wheel: limit lower=0 upper=0 effort=0 velocity=0 -> effort=30 velocity=100
- joint j_rear_right_wheel: limit lower=0 upper=0 effort=0 velocity=0 -> effort=30 velocity=100
- joint j_support_left: limit lower=0 upper=0 effort=0 velocity=0 -> lower=-1.0472 upper=1.0472 effort=10 velocity=100; type continuous -> revolute
- joint j_support_right: limit lower=0 upper=0 effort=0 velocity=0 -> lower=-1.0472 upper=1.0472 effort=30 velocity=100; type continuous -> revolute

File: urdf/robot_urdf.urdf (robot description, URDF)
Before this commit: robot robot_urdf, 7 links, 6 joints
Joints:
- joint j_front_left_wheel: limit lower=0 upper=0 effort=0 velocity=0 -> effort=30 velocity=100
- joint j_front_right_wheel: limit lower=0 upper=0 effort=0 velocity=0 -> effort=30 velocity=100
- joint j_rear_right_wheel: limit lower=0 upper=0 effort=0 velocity=0 -> effort=30 velocity=100
- joint j_support_left: limit lower=0 upper=0 effort=0 velocity=0 -> lower=-1.0472 upper=1.0472 effort=10 velocity=100; type continuous -> revolute
- joint j_support_right: limit lower=0 upper=0 effort=0 velocity=0 -> lower=-1.0472 upper=1.0472 effort=30 velocity=100; type continuous -> revolute

File: xacro/robot.xacro (robot description, xacro)
@@ -45,11 +45,11 @@
 	</gazebo>
 <!--  Gazebo plugin for control here is already added for you -->
-	<!-- <gazebo>
+	<gazebo>
 		<plugin name="gazebo_ros_control" filename="libgazebo_ros_control.so">
-			<robotNamespace>/robot_urdf</robotNamespace>
+			<robotNamespace>/robot_urdf/</robotNamespace>
 			<robotSimType>gazebo_ros_control/DefaultRobotHWSim</robotSimType>
 			<legacyModeNS>true</legacyModeNS>
 		</plugin>
-	</gazebo> -->
+	</gazebo>
 <!-- Create a joint between your robot and sensor -->
 	<joint

Commit message: Modified CAD designs, Added readme
touched up world files for better spawn camera position
added names to rviz and gazebo files which make sense
added README
tuned PID gains for effort controllers

File: urdf/integrated2.urdf (robot description, URDF)
Before this commit: robot robot_urdf, 10 links, 9 joints
Links:
- link base_link: mass 51.1408666026729 -> 51.2225965563684
- link front_left_wheel: mass 5.71507847538447 -> 0.737916384214473
- link front_right_wheel: mass 5.71507847538445 -> 0.737916384214473
- link rear_left_wheel: mass 5.71507847538444 -> 0.737916384214473
- link rear_right_wheel: mass 5.71507847538442 -> 0.737916384214473
- link support_left: mass 0.141762199312228 -> 0.511568168116717
- link support_right: mass 0.141762199312228 -> 0.511568168116718
Joints:
- joint j_front_left_wheel: axis 0 0 -1 -> 0 -1 0; origin xyz=0 -0.0299999999999973 -0.14732 rpy=1.5707963267949 0 0 -> xyz=0 0.03048 -0.14732 rpy=0 0 0
- joint j_front_right_wheel: axis 0 0 -1 -> 0 -1 0; origin xyz=0 -0.0299999999999997 -0.14732 rpy=1.5707963267949 0 0 -> xyz=0 -0.03048 -0.14732 rpy=0 0 0
- joint j_rear_left_wheel: axis 0 0 1 -> 0 -1 0; limit (none) -> effort=30 velocity=100; origin xyz=-0.3683 0.18113 0.11557 rpy=1.5707963267949 0 0 -> xyz=-0.381 0.18161 0.10211 rpy=0 0 0
- joint j_rear_right_wheel: axis 0 0 1 -> 0 -1 0; origin xyz=-0.3683 -0.18113 0.11557 rpy=1.5707963267949 0 0 -> xyz=-0.381 -0.18161 0.10211 rpy=0 0 0
- joint j_support_left: origin xyz=0.368299999999998 0.152399999999998 0.26289 rpy=0 0 0 -> xyz=0.3683 0.15113 0.24943 rpy=0 0 0
- joint j_support_right: limit lower=-1.0472 upper=1.0472 effort=30 velocity=100 -> lower=-1.0472 upper=1.0472 effort=10 velocity=100; origin xyz=0.3683 -0.1524 0.26289 rpy=0 0 0 -> xyz=0.3683 -0.15113 0.24943 rpy=0 0 0
- joint sensor_joint: origin xyz=0.44 0 0.275 rpy=0 0 0 -> xyz=0.45 0 0.265 rpy=0 0 0

File: urdf/robot_urdf.urdf (robot description, URDF)
Before this commit: robot robot_urdf, 7 links, 6 joints
Links:
- link base_link: mass 51.1408666026729 -> 51.2225965563684
- link front_left_wheel: mass 5.71507847538447 -> 0.737916384214473
- link front_right_wheel: mass 5.71507847538445 -> 0.737916384214473
- link rear_left_wheel: mass 5.71507847538444 -> 0.737916384214473
- link rear_right_wheel: mass 5.71507847538442 -> 0.737916384214473
- link support_left: mass 0.141762199312228 -> 0.511568168116717
- link support_right: mass 0.141762199312228 -> 0.511568168116718
Joints:
- joint j_front_left_wheel: axis 0 0 -1 -> 0 -1 0; origin xyz=0 -0.0299999999999973 -0.14732 rpy=1.5707963267949 0 0 -> xyz=0 0.03048 -0.14732 rpy=0 0 0
- joint j_front_right_wheel: axis 0 0 -1 -> 0 -1 0; origin xyz=0 -0.0299999999999997 -0.14732 rpy=1.5707963267949 0 0 -> xyz=0 -0.03048 -0.14732 rpy=0 0 0
- joint j_rear_left_wheel: axis 0 0 1 -> 0 -1 0; origin xyz=-0.3683 0.18113 0.11557 rpy=1.5707963267949 0 0 -> xyz=-0.381 0.18161 0.10211 rpy=0 0 0
- joint j_rear_right_wheel: axis 0 0 1 -> 0 -1 0; origin xyz=-0.3683 -0.18113 0.11557 rpy=1.5707963267949 0 0 -> xyz=-0.381 -0.18161 0.10211 rpy=0 0 0
- joint j_support_left: origin xyz=0.368299999999998 0.152399999999998 0.26289 rpy=0 0 0 -> xyz=0.3683 0.15113 0.24943 rpy=0 0 0
- joint j_support_right: origin xyz=0.3683 -0.1524 0.26289 rpy=0 0 0 -> xyz=0.3683 -0.15113 0.24943 rpy=0 0 0

File: xacro/robot.xacro (robot description, xacro)
@@ -57,5 +57,5 @@
       type="fixed">
 	  <origin
-		  xyz="0.44 0 0.275"
+		  xyz="0.45 0 0.265"
 		  rpy="0 0 0" />
     <parent
@@ -100,3 +100,39 @@
 		<child link="base_link"/>
 	</joint>
+	<transmission name="rear_drive_left">
+		<type>transmission_interface/SimpleTransmission</type>
+		<joint name="j_rear_left_wheel">
+			<hardwareInterface>hardware_interface/VelocityJointInterface</hardwareInterface>
+		</joint>
+		<actuator name="rear_motor_left">
+			<mechanicalReduction>1</mechanicalReduction>
+		</actuator>
+	</transmission>
+	<transmission name="rear_drive_right">
+		<type>transmission_interface/SimpleTransmission</type>
+		<joint name="j_rear_right_wheel">
+			<hardwareInterface>hardware_interface/VelocityJointInterface</hardwareInterface>
+		</joint>
+			<actuator name="rear_motor_right">
+		<mechanicalReduction>1</mechanicalReduction>
+		</actuator>
+	</transmission>
+	<transmission name="front_steering_left">
+		<type>transmission_interface/SimpleTransmission</type>
+		<joint name="j_support_left">
+			<hardwareInterface>hardware_interface/EffortJointInterface</hardwareInterface>
+		</joint>
+		<actuator name="front_motor_left">
+			<mechanicalReduction>1</mechanicalReduction>
+		</actuator>
+	</transmission>
+	<transmission name="front_steering_right">
+		<type>transmission_interface/SimpleTransmission</type>
+		<joint name="j_support_right">
+			<hardwareInterface>hardware_interface/EffortJointInterface</hardwareInterface>
+		</joint>
+		<actuator name="front_motor_right">
+			<mechanicalReduction>1</mechanicalReduction>
+		</actuator>
+	</transmission>
 </robot>

Commit message: Final Commit, Project Finished!

File: urdf/integrated2.urdf (robot description, URDF)
Before this commit: robot robot_urdf, 10 links, 9 joints
Links:
- link base_link: mass 51.2225965563684 -> 21.354
- link front_left_wheel: mass 0.737916384214473 -> 0.73792
- link front_right_wheel: mass 0.737916384214473 -> 0.73792
- link rear_left_wheel: mass 0.737916384214473 -> 0.73792
- link rear_right_wheel: mass 0.737916384214473 -> 0.73792
- link support_left: mass 0.511568168116717 -> 0.51157
- link support_right: mass 0.511568168116718 -> 0.51157
Joints:
- joint j_front_left_wheel: origin xyz=0 0.03048 -0.14732 rpy=0 0 0 -> xyz=0 0.03048 -0.13462 rpy=0 0 0
- joint j_front_right_wheel: origin xyz=0 -0.03048 -0.14732 rpy=0 0 0 -> xyz=0 -0.03048 -0.13462 rpy=0 0 0
- joint j_rear_left_wheel: origin xyz=-0.381 0.18161 0.10211 rpy=0 0 0 -> xyz=-0.26061 0.18161 0.1016 rpy=0 0 0
- joint j_rear_right_wheel: origin xyz=-0.381 -0.18161 0.10211 rpy=0 0 0 -> xyz=-0.26061 -0.18161 0.1016 rpy=0 0 0
- joint j_support_left: origin xyz=0.3683 0.15113 0.24943 rpy=0 0 0 -> xyz=0.2474 0.15113 0.23622 rpy=0 0 0
- joint j_support_right: origin xyz=0.3683 -0.15113 0.24943 rpy=0 0 0 -> xyz=0.2474 -0.15113 0.23622 rpy=0 0 0
- joint sensor_joint: origin xyz=0.45 0 0.265 rpy=0 0 0 -> xyz=0.525 0 0.2375 rpy=0 0 0

File: urdf/robot_urdf.urdf (robot description, URDF)
Before this commit: robot robot_urdf, 7 links, 6 joints
Links:
- link base_link: mass 51.2225965563684 -> 21.354
- link front_left_wheel: mass 0.737916384214473 -> 0.73792
- link front_right_wheel: mass 0.737916384214473 -> 0.73792
- link rear_left_wheel: mass 0.737916384214473 -> 0.73792
- link rear_right_wheel: mass 0.737916384214473 -> 0.73792
- link support_left: mass 0.511568168116717 -> 0.51157
- link support_right: mass 0.511568168116718 -> 0.51157
Joints:
- joint j_front_left_wheel: origin xyz=0 0.03048 -0.14732 rpy=0 0 0 -> xyz=0 0.03048 -0.13462 rpy=0 0 0
- joint j_front_right_wheel: origin xyz=0 -0.03048 -0.14732 rpy=0 0 0 -> xyz=0 -0.03048 -0.13462 rpy=0 0 0
- joint j_rear_left_wheel: origin xyz=-0.381 0.18161 0.10211 rpy=0 0 0 -> xyz=-0.26061 0.18161 0.1016 rpy=0 0 0
- joint j_rear_right_wheel: origin xyz=-0.381 -0.18161 0.10211 rpy=0 0 0 -> xyz=-0.26061 -0.18161 0.1016 rpy=0 0 0
- joint j_support_left: origin xyz=0.3683 0.15113 0.24943 rpy=0 0 0 -> xyz=0.2474 0.15113 0.23622 rpy=0 0 0
- joint j_support_right: origin xyz=0.3683 -0.15113 0.24943 rpy=0 0 0 -> xyz=0.2474 -0.15113 0.23622 rpy=0 0 0

File: xacro/robot.xacro (robot description, xacro)
@@ -57,5 +57,5 @@
       type="fixed">
 	  <origin
-		  xyz="0.45 0 0.265"
+		  xyz="0.525 0 0.2375"
 		  rpy="0 0 0" />
     <parent
@@ -74,23 +74,23 @@
 	</material>
 	<gazebo reference="base_link">
-		<material>Gazebo/Red</material>
+		<material>Gazebo/SkyBlue</material>
 	</gazebo>
 	<gazebo reference="support_left">
-		<material>Gazebo/Red</material>
+		<material>Gazebo/SkyBlue</material>
 	</gazebo>
 	<gazebo reference="support_right">
-		<material>Gazebo/Red</material>
+		<material>Gazebo/SkyBlue</material>
 	</gazebo>
 	<gazebo reference="front_left_wheel">
-		<material>Gazebo/FlatBlack</material>
+		<material>Gazebo/Grey</material>
 	</gazebo>
 	<gazebo reference="front_right_wheel">
-		<material>Gazebo/FlatBlack</material>
+		<material>Gazebo/Grey</material>
 	</gazebo>
 	<gazebo reference="rear_left_wheel">
-		<material>Gazebo/FlatBlack</material>
+		<material>Gazebo/Grey</material>
 	</gazebo>
 	<gazebo reference="rear_right_wheel">
-		<material>Gazebo/FlatBlack</material>
+		<material>Gazebo/Grey</material>
 	</gazebo>
 	<link name="dummy_link">
